File: eagle/BeebOPL.brd (EAGLE design)
At the start: 100 x 80 mm, 46 parts, among them IC1 LM324N, IC2 YM3014B, IC3 LM7805, IC5 74LS02N, IC6 YM3812, IC7 74LS04N, IC9 74HCT688N, J1 1 MHz Bus, J2 Feed-through, J3 3.5mm Jack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

Commit message: Further refined schematic
Parts:
- added C10, C11: 10nF, resistor:C050-024X044
- JP3: value (none) -> AUDIO
- JP4: value (none) -> LED
- JP5: value (none) -> PWR
- S2: device SparkFun-Retired:1X02 -> SparkFun-Retired:SJ_2S-TRACE-PTH
- S3: value (none) -> REG; device SparkFun-Retired:1X03 -> YMSynth:S_3WAY_OR
- TR1: value IRFD9024DIL -> IRFD9024; device YMSynth:FET-DIL -> YMSynth:FET-DIL-OPTN
- moved S2 246.5 mm to (-32.6, -169.3)
- moved S3 61.8 mm to (-32.6, -172.3)
- moved TR1 60.7 mm to (-29.8, -178.9)
Connections:
- new net N$29: S3.1, TR1.S
- new net N$4: J4.PWR, JP5.4, TR1.D, TR1.D1
- new net YM/IRQ: IC6./IRQ, S2.2
- net /IRQ: no longer IC6./IRQ, S2.2
- net GND: now also C10.2, C11.2
- net VCC: now also C10.1, C11.1; no longer J4.PWR, JP5.4, S3.1, TR1.D, TR1.D1, TR1.S
Routing:
- net YM/IRQ: track 0.00 -> 48.5 mm
- net /IRQ: track 93.7 -> 45.1 mm
Changed lines of the file:
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@@
 <attribute name="VALUE" x="13.335" y="72.898" size="1.27" layer="27"/>
-</element>
-<element name="S2" library="SparkFun-Retired" package="1X02" value="IRQ" x="40.64" y="66.04" smashed="yes">
-<attribute name="NAME" x="40.5638" y="67.8688" size="1.27" layer="25" ratio="10"/>
-<attribute name="VALUE" x="40.005" y="62.865" size="1.27" layer="27"/>
 </element>
 <element name="R7" library="resistor" package="0207/10" value="470R" x="82.55" y="21.59" smashed="yes">
@@
 <element name="R9" library="resistor" package="0207/10" value="470R" x="0.127" y="-104.521"/>
 <element name="IC3" library="linear" package="TO220V" value="LM7805" x="-0.508" y="-105.791"/>
-<element name="S3" library="SparkFun-Retired" package="1X03" value="" x="-4.191" y="-117.475"/>
-<element name="TR1" library="YMSynth" package="FET-DIL" value="IRFD9024DIL" x="-0.127" y="-125.984"/>
-<element name="JP3" library="pinhead" package="1X02/90" value="" x="-20.955" y="-124.841"/>
-<element name="JP4" library="pinhead" package="1X02/90" value="" x="-30.861" y="-124.841"/>
-<element name="JP5" library="pinhead" package="1X04/90" value="" x="-28.321" y="-138.176"/>
+<element name="JP3" library="pinhead" package="1X02/90" value="AUDIO" x="-20.955" y="-124.841"/>
+<element name="JP4" library="pinhead" package="1X02/90" value="LED" x="-30.861" y="-124.841"/>
+<element name="JP5" library="pinhead" package="1X04/90" value="PWR" x="-28.321" y="-138.176"/>
+<element name="C10" library="resistor" package="C050-024X044" value="10nF" x="-32.131" y="-158.496"/>
+<element name="C11" library="resistor" package="C050-024X044" value="10nF" x="-32.131" y="-164.846"/>
+<element name="S2" library="SparkFun-Retired" package="SJ_2S-TRACE-PTH" value="IRQ" x="-32.639" y="-169.291"/>
+<element name="S3" library="YMSynth" package="S_3WAY_OR" value="REG" x="-32.639" y="-172.339"/>
+<element name="TR1" library="YMSynth" package="FET-DIL-OPTN" value="IRFD9024" x="-29.845" y="-178.943"/>
 </elements>
 <signals>
@@
 <contactref element="JP3" pad="2"/>
 <contactref element="JP4" pad="2"/>
-<contactref element="TR1" pad="G"/>
 <contactref element="IC9" pad="3"/>
 <contactref element="IC9" pad="5"/>
 <contactref element="JP5" pad="2"/>
 <contactref element="JP5" pad="3"/>
+<contactref element="C10" pad="2"/>
+<contactref element="C11" pad="2"/>
+<contactref element="TR1" pad="G"/>
+<wire x1="-29.591" y1="-164.846" x2="-26.035" y2="-180.213" width="0" layer="19" extent="1-1"/>
+<wire x1="-29.591" y1="-158.496" x2="-29.591" y2="-164.846" width="0" layer="19" extent="1-1"/>
+<wire x1="-29.591" y1="-141.986" x2="-29.591" y2="-158.496" width="0" layer="19" extent="1-1"/>
 <wire x1="-27.051" y1="-141.986" x2="-29.591" y2="-141.986" width="0" layer="19" extent="1-1"/>
 <wire x1="-29.591" y1="-128.651" x2="-29.591" y2="-141.986" width="0" layer="19" extent="1-1"/>
 <wire x1="-19.685" y1="-128.651" x2="-29.591" y2="-128.651" width="0" layer="19" extent="1-1"/>
-<wire x1="3.683" y1="-127.254" x2="-19.685" y2="-128.651" width="0" layer="19" extent="1-1"/>
-<wire x1="-0.508" y1="-108.331" x2="3.683" y2="-127.254" width="0" layer="19" extent="1-1"/>
+<wire x1="-0.508" y1="-108.331" x2="-19.685" y2="-128.651" width="0" layer="19" extent="1-1"/>
 <wire x1="-1.524" y1="-97.917" x2="-0.508" y2="-108.331" width="0" layer="19" extent="1-1"/>
 <wire x1="-3.302" y1="-85.344" x2="-1.524" y2="-97.917" width="0" layer="19" extent="1-1"/>
@@
 <wire x1="15.494" y1="16.51" x2="21.59" y2="16.51" width="1.016" layer="16"/>
 <wire x1="13.97" y1="14.986" x2="15.494" y2="16.51" width="1.016" layer="16"/>
+<contactref element="IC9" pad="7"/>
+<contactref element="C10" pad="1"/>
+<contactref element="C11" pad="1"/>
 <contactref element="S3" pad="2"/>
-<contactref element="S3" pad="1"/>
-<contactref element="TR1" pad="S"/>
-<contactref element="J4" pad="PWR"/>
-<contactref element="TR1" pad="D1"/>
-<contactref element="TR1" pad="D"/>
-<contactref element="IC9" pad="7"/>
-<contactref element="JP5" pad="4"/>
-<wire x1="-3.937" y1="-127.254" x2="-24.511" y2="-141.986" width="0" layer="19" extent="1-1"/>
-<wire x1="-3.937" y1="-124.714" x2="-3.937" y2="-127.254" width="0" layer="19" extent="1-1"/>
-<wire x1="-4.191" y1="-117.475" x2="-3.937" y2="-124.714" width="0" layer="19" extent="1-1"/>
-<wire x1="-1.651" y1="-117.475" x2="-4.191" y2="-117.475" width="0" layer="19" extent="1-1"/>
-<wire x1="3.683" y1="-124.714" x2="-3.937" y2="-124.714" width="0" layer="19" extent="1-1"/>
-<wire x1="2.032" y1="-108.331" x2="-1.651" y2="-117.475" width="0" layer="19" extent="1-1"/>
+<wire x1="-34.671" y1="-164.846" x2="-31.369" y2="-172.339" width="0" layer="19" extent="1-1"/>
+<wire x1="-34.671" y1="-158.496" x2="-34.671" y2="-164.846" width="0" layer="19" extent="1-1"/>
+<wire x1="2.032" y1="-108.331" x2="-34.671" y2="-158.496" width="0" layer="19" extent="1-1"/>
 <wire x1="5.207" y1="-104.521" x2="2.032" y2="-108.331" width="0" layer="19" extent="1-1"/>
 <wire x1="-3.302" y1="-80.264" x2="5.207" y2="-104.521" width="0" layer="19" extent="1-1"/>
@@
 <wire x1="12.573" y1="-24.257" x2="-3.302" y2="-70.104" width="0" layer="19" extent="1-1"/>
 <wire x1="-2.667" y1="-16.637" x2="12.573" y2="-24.257" width="0" layer="19" extent="1-1"/>
-<wire x1="8.72" y1="16.47" x2="-2.667" y2="-16.637" width="0" layer="19" extent="1-1"/>
-<wire x1="13.97" y1="14.986" x2="8.72" y2="16.47" width="0" layer="19" extent="1-1"/>
+<wire x1="13.97" y1="14.986" x2="-2.667" y2="-16.637" width="0" layer="19" extent="1-1"/>
 <wire x1="30.988" y1="16.51" x2="21.59" y2="16.51" width="0" layer="19" extent="1-1"/>
 <wire x1="82.677" y1="31.75" x2="93.98" y2="19.05" width="0" layer="19" extent="1-16"/>
@@
 <wire x1="48.641" y1="79.375" x2="51.562" y2="79.375" width="0.2286" layer="1"/>
 <wire x1="51.562" y1="79.375" x2="52.959" y2="77.978" width="0.2286" layer="1"/>
-<contactref element="S2" pad="2"/>
 <contactref element="S2" pad="1"/>
-<contactref element="IC6" pad="/IRQ"/>
-<wire x1="40.64" y1="64.262" x2="49.5935" y2="55.3085" width="0.254" layer="16"/>
-<wire x1="57.15" y1="24.13" x2="59.055" y2="26.035" width="0.254" layer="16"/>
-<wire x1="59.055" y1="26.035" x2="59.055" y2="31.115" width="0.254" layer="16"/>
-<wire x1="59.055" y1="31.115" x2="52.07" y2="38.1" width="0.254" layer="16"/>
-<wire x1="52.07" y1="38.1" x2="52.07" y2="46.355" width="0.254" layer="16"/>
-<wire x1="52.07" y1="46.355" x2="49.5935" y2="48.8315" width="0.254" layer="16"/>
-<wire x1="49.5935" y1="48.8315" x2="49.5935" y2="55.3085" width="0.254" layer="16"/>
-<wire x1="43.18" y1="66.04" x2="46.99" y2="69.85" width="0" layer="19" extent="16-16"/>
-<wire x1="44.831" y1="64.389" x2="43.18" y2="66.04" width="0" layer="19" extent="16-16"/>
-<wire x1="40.64" y1="66.04" x2="43.18" y2="66.04" width="0" layer="19" extent="1-1"/>
-<wire x1="40.64" y1="64.262" x2="40.64" y2="66.04" width="0" layer="19" extent="16-16"/>
+<wire x1="48.133" y1="59.69" x2="-33.909" y2="-169.291" width="0" layer="19" extent="16-16"/>
+<wire x1="46.99" y1="69.85" x2="44.831" y2="64.389" width="0" layer="19" extent="16-16"/>
 </signal>
 <signal name="/NMI">
@@
 </signal>
 <signal name="N$27">
+<contactref element="IC3" pad="1"/>
 <contactref element="S3" pad="3"/>
-<contactref element="IC3" pad="1"/>
-<wire x1="-3.048" y1="-108.331" x2="0.889" y2="-117.475" width="0" layer="19" extent="1-1"/>
+<wire x1="-3.048" y1="-108.331" x2="-28.829" y2="-172.339" width="0" layer="19" extent="1-1"/>
 </signal>
 <signal name="N$26">
@@
 <wire x1="80.01" y1="6.604" x2="80.01" y2="8.89" width="0" layer="19" extent="1-1"/>
 </signal>
+<signal name="N$4" class="1">
+<contactref element="J4" pad="PWR"/>
+<contactref element="JP5" pad="4"/>
+<contactref element="TR1" pad="D"/>
+<contactref element="TR1" pad="D1"/>
+<wire x1="-33.655" y1="-177.673" x2="-33.655" y2="-180.213" width="0" layer="19" extent="1-1"/>
+<wire x1="-24.511" y1="-141.986" x2="-33.655" y2="-177.673" width="0" layer="19" extent="1-1"/>
+<wire x1="8.72" y1="16.47" x2="-24.511" y2="-141.986" width="0" layer="19" extent="1-1"/>
+</signal>
+<signal name="N$29" class="1">
+<contactref element="S3" pad="1"/>
+<contactref element="TR1" pad="S"/>
+<wire x1="-26.035" y1="-177.673" x2="-33.909" y2="-172.339" width="0" layer="19" extent="1-1"/>
+</signal>
+<signal name="YM/IRQ">
+<contactref element="IC6" pad="/IRQ"/>
+<wire x1="40.64" y1="64.262" x2="49.5935" y2="55.3085" width="0.254" layer="16"/>
+<wire x1="57.15" y1="24.13" x2="59.055" y2="26.035" width="0.254" layer="16"/>
+<wire x1="59.055" y1="26.035" x2="59.055" y2="31.115" width="0.254" layer="16"/>
+<wire x1="59.055" y1="31.115" x2="52.07" y2="38.1" width="0.254" layer="16"/>
+<wire x1="52.07" y1="38.1" x2="52.07" y2="46.355" width="0.254" layer="16"/>
+<wire x1="52.07" y1="46.355" x2="49.5935" y2="48.8315" width="0.254" layer="16"/>
+<wire x1="49.5935" y1="48.8315" x2="49.5935" y2="55.3085" width="0.254" layer="16"/>
+<contactref element="S2" pad="2"/>
+<wire x1="57.15" y1="24.13" x2="-31.369" y2="-169.291" width="0" layer="19" extent="1-1"/>
+</signal>
 </signals>

Commit message: More sophisticated power section
Parts:
- J4: value 5V DC -> DC-IN
- moved S3 271.1 mm to (-55.9, 97.8)
- moved S2 268.7 mm to (-62.2, 97.8)
- moved C11 246.6 mm to (-16.5, 81.3)
- moved TR1 245.5 mm to (-59.7, 64.8)
- moved C10 239.0 mm to (-88.9, 73.7)
- moved R9 207.2 mm to (-44.5, 97.8)
- moved RN4 191.9 mm to (-76.2, 87.6)
- moved IC3 188.1 mm to (-71.1, 68.6)
- moved XTAL1 185.3 mm to (-82.5, 64.8), turned to 0 degrees
- moved C9 185.1 mm to (-81.3, 73.7), turned to 0 degrees
- moved RN3 177.5 mm to (-50.8, 87.6)
- moved LED1 174.7 mm to (-35.6, 73.7)
- moved RN1 170.9 mm to (-74.9, 80.0)
- moved RN2 166.0 mm to (-25.4, 87.6)
- moved JP4 152.1 mm to (-17.8, 26.7)
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Connections:
- removed net N$27: IC3.1, S3.3
- new net +12V: IC3.1, JP5.1, S3.3
- new net +5V: IC3.3, JP5.4, S3.1, TR1.D, TR1.D1
- net GND: no longer JP5.2, JP5.3
- net N$29: now also JP5.2, JP5.3; no longer S3.1, TR1.S
- net N$4: now also S3.2; no longer JP5.4, TR1.D, TR1.D1
- net VCC: now also TR1.S; no longer IC3.3, S3.2
Routing:
- net GND: track 343.0 -> 0.00 mm, vias 3 -> 0
- net D4: track 180.2 -> 0.00 mm, vias 1 -> 0
- net VCC: track 171.2 -> 0.00 mm, vias 4 -> 0
- net D2: track 156.1 -> 0.00 mm, vias 5 -> 0
- net D6: track 132.0 -> 0.00 mm, vias 3 -> 0
- net D7: track 129.2 -> 0.00 mm
- net D3: track 115.9 -> 0.00 mm, vias 3 -> 0
- net D5: track 107.1 -> 0.00 mm, vias 1 -> 0
- net /RST: track 105.5 -> 0.00 mm, vias 5 -> 0
- net N$7: track 103.4 -> 0.00 mm, vias 2 -> 0
- net N$11: track 102.4 -> 0.00 mm, vias 2 -> 0
- net 1MHZE: track 95.9 -> 0.00 mm, vias 3 -> 0
- net /PGFC: track 92.6 -> 0.00 mm, vias 2 -> 0
- net D0: track 86.3 -> 0.00 mm, vias 3 -> 0
- net D1: track 86.0 -> 0.00 mm, vias 1 -> 0
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- removed copper zone on layer 1, net GND
- removed copper zone on layer 16, net GND
Other:
- board text removed: "BeebOPL"

Commit message: Assigned net classes
Connections:
- net N$17 renamed AUDIO_OUT
- net N$4 renamed DC
- removed net N$29: JP5.2, JP5.3
- net GND: now also JP5.2, JP5.3
Changed lines of the file:
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@@
 <contactref element="C11" pad="2"/>
 <contactref element="C6" pad="-"/>
-<wire x1="-81.28" y1="24.13" x2="-80.01" y2="2.54" width="0" layer="19" extent="1-1"/>
+<contactref element="JP5" pad="3"/>
+<contactref element="JP5" pad="2"/>
+<wire x1="-69.85" y1="2.54" x2="-80.01" y2="2.54" width="0" layer="19" extent="1-1"/>
+<wire x1="-67.31" y1="2.54" x2="-69.85" y2="2.54" width="0" layer="19" extent="1-1"/>
+<wire x1="-50.84" y1="12.07" x2="-67.31" y2="2.54" width="0" layer="19" extent="1-1"/>
+<wire x1="-53.34" y1="26.67" x2="-50.84" y2="12.07" width="0" layer="19" extent="1-1"/>
+<wire x1="-63.5" y1="24.13" x2="-53.34" y2="26.67" width="0" layer="19" extent="1-1"/>
+<wire x1="-66.04" y1="24.13" x2="-63.5" y2="24.13" width="0" layer="19" extent="1-1"/>
+<wire x1="-68.58" y1="24.13" x2="-66.04" y2="24.13" width="0" layer="19" extent="1-1"/>
+<wire x1="-71.12" y1="24.13" x2="-68.58" y2="24.13" width="0" layer="19" extent="1-1"/>
+<wire x1="-73.66" y1="24.13" x2="-71.12" y2="24.13" width="0" layer="19" extent="1-1"/>
+<wire x1="-76.2" y1="24.13" x2="-73.66" y2="24.13" width="0" layer="19" extent="1-1"/>
+<wire x1="-78.74" y1="24.13" x2="-76.2" y2="24.13" width="0" layer="19" extent="1-1"/>
+<wire x1="-81.28" y1="24.13" x2="-78.74" y2="24.13" width="0" layer="19" extent="1-1"/>
 <wire x1="-83.82" y1="24.13" x2="-81.28" y2="24.13" width="0" layer="19" extent="1-1"/>
-<wire x1="-78.74" y1="24.13" x2="-81.28" y2="24.13" width="0" layer="19" extent="1-1"/>
-<wire x1="-76.2" y1="24.13" x2="-78.74" y2="24.13" width="0" layer="19" extent="1-1"/>
-<wire x1="-73.66" y1="24.13" x2="-76.2" y2="24.13" width="0" layer="19" extent="1-1"/>
-<wire x1="-71.12" y1="24.13" x2="-73.66" y2="24.13" width="0" layer="19" extent="1-1"/>
-<wire x1="-68.58" y1="24.13" x2="-71.12" y2="24.13" width="0" layer="19" extent="1-1"/>
-<wire x1="-66.04" y1="24.13" x2="-68.58" y2="24.13" width="0" layer="19" extent="1-1"/>
-<wire x1="-63.5" y1="24.13" x2="-66.04" y2="24.13" width="0" layer="19" extent="1-1"/>
-<wire x1="-53.34" y1="26.67" x2="-63.5" y2="24.13" width="0" layer="19" extent="1-1"/>
 <wire x1="-54.61" y1="38.1" x2="-53.34" y2="26.67" width="0" layer="19" extent="1-1"/>
 <wire x1="-57.15" y1="38.1" x2="-54.61" y2="38.1" width="0" layer="19" extent="1-1"/>
@@
 <wire x1="-30.48" y1="26.67" x2="-29.21" y2="40.64" width="0" layer="19" extent="1-1"/>
 <wire x1="-16.51" y1="22.86" x2="-30.48" y2="26.67" width="0" layer="19" extent="1-1"/>
-<wire x1="-50.84" y1="12.07" x2="-53.34" y2="26.67" width="0" layer="19" extent="1-1"/>
 <wire x1="-22.86" y1="57.15" x2="-35.56" y2="49.53" width="0" layer="19" extent="1-1"/>
 <wire x1="-86.36" y1="73.66" x2="-71.12" y2="73.66" width="0" layer="19" extent="1-1"/>
@@
 <wire x1="-15.24" y1="49.53" x2="-32.766" y2="80.01" width="0" layer="19" extent="1-1"/>
 </signal>
-<signal name="N$17" class="2">
+<signal name="AUDIO_OUT" class="2">
 <contactref element="C1" pad="-"/>
 <contactref element="J3" pad="TIP"/>
@@
 <wire x1="-60.96" y1="97.79" x2="-39.37" y2="2.54" width="0" layer="19" extent="1-1"/>
 </signal>
-<signal name="+12V">
+<signal name="+12V" class="1">
 <contactref element="JP5" pad="1"/>
 <contactref element="IC3" pad="1"/>
@@
 <wire x1="-57.15" y1="97.79" x2="-63.5" y2="66.04" width="0" layer="19" extent="1-1"/>
 </signal>
-<signal name="N$4">
+<signal name="DC" class="1">
 <contactref element="J4" pad="PWR"/>
 <contactref element="S3" pad="2"/>
 <wire x1="-55.84" y1="15.07" x2="-54.61" y2="97.79" width="0" layer="19" extent="1-1"/>
 </signal>
-<signal name="N$29">
-<contactref element="JP5" pad="2"/>
-<contactref element="JP5" pad="3"/>
-<wire x1="-67.31" y1="2.54" x2="-69.85" y2="2.54" width="0" layer="19" extent="1-1"/>
-</signal>
 </signals>

Commit message: Initial board layout
Parts:
- removed H1, H2, H3, H4: MOUNT-HOLE4.1, holes:4,1
- JP3, JP4: device pinhead:1X02/90 -> pinhead:1X02
- JP5: device pinhead:1X04/90 -> pinhead:1X04
- LED1: value (none) -> LED
- moved C10 189.4 mm to (95.2, 29.2), turned to 180 degrees
- moved XTAL1 184.6 mm to (95.2, 15.2), turned to 270 degrees
- moved C9 179.3 mm to (83.8, 3.81)
- moved RN4 168.2 mm to (87.6, 49.5)
- moved IC9 165.1 mm to (86.4, 39.4), turned to 180 degrees
- moved C8 153.8 mm to (68.6, 15.2), turned to 270 degrees
- moved C5 151.4 mm to (86.4, 29.2), turned to 180 degrees
- moved IC7 149.7 mm to (81.3, 15.2), turned to 180 degrees
- moved R8 146.6 mm to (83.8, 7.62), turned to 180 degrees
- moved RN3 142.6 mm to (87.6, 53.3)
- moved RN1 141.0 mm to (63.5, 53.3)
- moved J1 139.4 mm to (67.3, 73.7)
- moved R7 127.3 mm to (83.8, 22.9), turned to 180 degrees
- moved IC2 119.5 mm to (39.4, 48.3), turned to 180 degrees
- moved R6 118.8 mm to (21.6, 35.6), turned to 90 degrees
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Connections:
- net A1: now also IC9.11; no longer IC9.4
- net A2: now also IC9.8; no longer IC9.6
- net A3: now also IC9.13; no longer IC9.8
- net A4: now also IC9.6; no longer IC9.11
- net A5: now also IC9.15; no longer IC9.13
- net A6: now also IC9.4; no longer IC9.15
- net GND: now also IC9.7; no longer IC9.9
- net VCC: now also IC9.9; no longer IC9.7
Routing:
- net GND: track 0.00 -> 149.3 mm
- net A7: track 0.00 -> 48.5 mm
- net A5: track 0.00 -> 48.2 mm
- net A3: track 0.00 -> 46.2 mm
- net VCC: track 0.00 -> 44.1 mm
- net A1: track 0.00 -> 44.1 mm
- net A6: track 0.00 -> 37.8 mm
- net D0: track 0.00 -> 36.1 mm
- net A4: track 0.00 -> 35.7 mm
- net A2: track 0.00 -> 33.9 mm
- net D2: track 0.00 -> 33.8 mm
- net /PGFC: track 0.00 -> 33.1 mm
- net D1: track 0.00 -> 32.2 mm
- net N$1: track 0.00 -> 31.8 mm
- net D4: track 0.00 -> 31.5 mm
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
Commit message: Routing signals
Parts:
- C10, C11: value 10nF -> 100nF
- moved S2 9.67 mm to (34.3, 76.2)
- moved C1 6.84 mm to (21.6, 61.0)
- moved S1 4.02 mm to (14.0, 76.2)
- moved R1 1.27 mm to (22.9, 69.8)
- moved J3 1.27 mm to (3.81, 66.0)
- moved JP3 1.27 mm to (6.35, 55.9)
- turned R4 to 270 degrees
Connections:
- net GND: now also J4.GND@1
Routing:
- net GND: track 149.3 -> 386.2 mm, vias 0 -> 2
- net VCC: track 44.1 -> 180.6 mm, vias 0 -> 1
- net N$23: track 0.00 -> 64.7 mm, vias 0 -> 3
- net D5: track 27.5 -> 87.6 mm
- net D7: track 25.5 -> 84.8 mm
- net D6: track 29.3 -> 88.6 mm
- net D4: track 31.5 -> 88.6 mm
- net D2: track 33.8 -> 90.9 mm
- net D3: track 29.8 -> 86.9 mm
- net CNPGFC: track 15.2 -> 61.2 mm, vias 0 -> 4
- net N$14: track 0.00 -> 35.0 mm
- net AUDIO_OUT: track 0.00 -> 34.7 mm
- net R/W: track 17.9 -> 49.5 mm, vias 0 -> 2
- net 1MHZE: track 17.9 -> 47.3 mm, vias 0 -> 2
- net N$15: track 0.00 -> 29.3 mm, vias 0 -> 1
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
Commit message: Further routing
Routing:
- net YM/IRQ: track 0.00 -> 88.6 mm, vias 0 -> 3
- net AUDIO: track 13.8 -> 64.1 mm
- net D1: track 32.2 -> 71.0 mm, vias 0 -> 2
- net GND: track 386.2 -> 423.5 mm
- net N$19: track 2.54 -> 36.9 mm
- net N$8: track 18.3 -> 45.6 mm, vias 0 -> 4
- net N$13: track 12.5 -> 39.6 mm
- net N$11: track 0.00 -> 24.1 mm
- net N$16: track 23.4 -> 44.0 mm
- net /IRQ: track 17.9 -> 38.0 mm
- net N$6: track 18.3 -> 37.5 mm, vias 0 -> 2
- net N$7: track 18.3 -> 36.4 mm, vias 0 -> 4
- net AUDIO_OUT: track 34.7 -> 37.2 mm
