File: eagle/BeebOPL.brd (EAGLE design)
At the start: 100 x 80 mm, 44 parts, among them IC1 LM324N, IC2 YM3014B, IC3 LM7805, IC5 74LS02N, IC6 YM3812, IC7 74LS04N, IC9 74HCT688N, J1 1 MHz Bus, J2 Feed-through, J3 3.5mm Jack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

Commit message: Manual routing not complete
Routing:
- net N$6: track 37.5 -> 0.00 mm, vias 2 -> 0
- net N$7: track 36.4 -> 0.00 mm, vias 4 -> 0
- net GND: track 423.5 -> 435.7 mm
- net N$8: track 45.6 -> 57.5 mm
Changed lines of the file:
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@@
 <wire x1="5.715" y1="73.025" x2="5.715" y2="67.945" width="1.016" layer="1"/>
 <wire x1="5.715" y1="67.945" x2="3.81" y2="66.04" width="1.016" layer="1"/>
-<wire x1="77.47" y1="49.53" x2="78.74" y2="58.42" width="0" layer="19" extent="16-16"/>
-<wire x1="82.55" y1="43.18" x2="77.47" y2="46.99" width="0" layer="19" extent="16-16"/>
-<wire x1="87.63" y1="35.56" x2="87.63" y2="41.275" width="0" layer="19" extent="1-1"/>
-<wire x1="67.31" y1="71.12" x2="77.47" y2="69.85" width="0" layer="19" extent="16-16"/>
+<wire x1="3.81" y1="66.04" x2="3.81" y2="64.77" width="1.016" layer="1"/>
+<wire x1="3.81" y1="64.77" x2="5.715" y2="62.865" width="1.016" layer="1"/>
+<wire x1="5.715" y1="62.865" x2="5.715" y2="56.515" width="1.016" layer="1"/>
+<wire x1="5.715" y1="56.515" x2="5.08" y2="55.88" width="1.016" layer="1"/>
+<wire x1="77.47" y1="49.53" x2="75.565" y2="49.53" width="1.016" layer="16"/>
+<wire x1="75.565" y1="49.53" x2="75.565" y2="55.245" width="1.016" layer="16"/>
+<wire x1="75.565" y1="55.245" x2="78.74" y2="58.42" width="1.016" layer="16"/>
 <wire x1="64.77" y1="71.12" x2="66.04" y2="69.85" width="0" layer="19" extent="16-16"/>
 <wire x1="62.23" y1="71.12" x2="63.5" y2="69.85" width="0" layer="19" extent="16-16"/>
@@
 <wire x1="46.99" y1="71.12" x2="48.26" y2="69.85" width="0" layer="19" extent="16-16"/>
 <wire x1="53.34" y1="49.53" x2="54.61" y2="58.42" width="0" layer="19" extent="16-16"/>
+<wire x1="75.565" y1="55.245" x2="67.31" y2="59.69" width="0" layer="19" extent="16-16"/>
+<wire x1="82.55" y1="43.18" x2="77.47" y2="46.99" width="0" layer="19" extent="16-16"/>
+<wire x1="87.63" y1="35.56" x2="87.63" y2="41.275" width="0" layer="19" extent="1-1"/>
 <wire x1="38.1" y1="44.45" x2="53.34" y2="43.18" width="0" layer="19" extent="1-1"/>
-<wire x1="5.08" y1="55.88" x2="22.86" y2="46.355" width="0" layer="19" extent="1-1"/>
-<wire x1="3.81" y1="66.04" x2="3.81" y2="64.77" width="1.016" layer="1"/>
-<wire x1="3.81" y1="64.77" x2="5.715" y2="62.865" width="1.016" layer="1"/>
-<wire x1="5.715" y1="62.865" x2="5.715" y2="56.515" width="1.016" layer="1"/>
-<wire x1="5.715" y1="56.515" x2="5.08" y2="55.88" width="1.016" layer="1"/>
+<wire x1="5.715" y1="56.515" x2="22.86" y2="46.355" width="0" layer="19" extent="1-1"/>
 </signal>
 <signal name="D0">
@@
 <contactref element="IC6" pad="SH"/>
 <contactref element="IC2" pad="LOAD"/>
-<wire x1="54.61" y1="7.62" x2="54.61" y2="15.875" width="0.254" layer="1"/>
-<wire x1="38.1" y1="52.07" x2="40.005" y2="50.165" width="0.254" layer="1"/>
-<wire x1="40.005" y1="50.165" x2="43.815" y2="50.165" width="0.254" layer="1"/>
-<wire x1="43.815" y1="50.165" x2="46.99" y2="46.99" width="0.254" layer="1"/>
-<wire x1="46.99" y1="29.845" x2="46.99" y2="45.72" width="0" layer="19" extent="1-16"/>
-<wire x1="48.26" y1="27.94" x2="46.99" y2="29.845" width="0.254" layer="16"/>
-<wire x1="48.26" y1="22.225" x2="48.26" y2="27.94" width="0.254" layer="16"/>
-<wire x1="50.8" y1="19.685" x2="48.26" y2="22.225" width="0.254" layer="16"/>
-<wire x1="46.99" y1="46.99" x2="46.99" y2="45.72" width="0.254" layer="1"/>
-<via x="46.99" y="45.72" extent="1-16" drill="0.6"/>
-<via x="50.8" y="19.685" extent="1-16" drill="0.6"/>
-<wire x1="50.8" y1="19.685" x2="54.61" y2="15.875" width="0.254" layer="1"/>
+<wire x1="54.61" y1="7.62" x2="38.1" y2="52.07" width="0" layer="19" extent="1-1"/>
 </signal>
 <signal name="N$7">
 <contactref element="IC6" pad="MO"/>
 <contactref element="IC2" pad="SD"/>
-<wire x1="57.15" y1="7.62" x2="57.15" y2="15.875" width="0.254" layer="1"/>
-<wire x1="35.56" y1="52.07" x2="35.56" y2="51.435" width="0.254" layer="1"/>
-<wire x1="35.56" y1="51.435" x2="40.005" y2="46.99" width="0.254" layer="1"/>
-<wire x1="40.005" y1="46.99" x2="43.18" y2="46.99" width="0.254" layer="1"/>
-<wire x1="43.18" y1="46.99" x2="45.085" y2="45.085" width="0.254" layer="1"/>
-<wire x1="45.085" y1="43.815" x2="45.085" y2="45.085" width="0.254" layer="1"/>
-<wire x1="45.72" y1="42.545" x2="45.085" y2="43.815" width="0" layer="19" extent="1-16"/>
-<wire x1="45.72" y1="22.225" x2="45.72" y2="42.545" width="0" layer="19" extent="1-16"/>
-<wire x1="50.8" y1="17.145" x2="45.72" y2="22.225" width="0.254" layer="16"/>
-<wire x1="52.07" y1="17.145" x2="50.8" y2="17.145" width="0.254" layer="1"/>
-<wire x1="53.34" y1="15.875" x2="52.07" y2="17.145" width="0.254" layer="1"/>
-<wire x1="57.15" y1="15.875" x2="53.34" y2="15.875" width="0.254" layer="16"/>
-<via x="45.085" y="43.815" extent="1-16" drill="0.6"/>
-<via x="50.8" y="17.145" extent="1-16" drill="0.6"/>
-<via x="53.34" y="15.875" extent="1-16" drill="0.6"/>
-<via x="57.15" y="15.875" extent="1-16" drill="0.6"/>
+<wire x1="57.15" y1="7.62" x2="35.56" y2="52.07" width="0" layer="19" extent="1-1"/>
 </signal>
 <signal name="N$8">
@@
 <wire x1="36.83" y1="38.735" x2="36.83" y2="43.18" width="0.254" layer="1"/>
 <wire x1="36.83" y1="29.845" x2="36.83" y2="38.735" width="0.254" layer="16"/>
-<wire x1="43.18" y1="23.495" x2="36.83" y2="29.845" width="0" layer="19" extent="1-16"/>
-<wire x1="43.18" y1="22.225" x2="43.18" y2="23.495" width="0.254" layer="16"/>
-<wire x1="50.8" y1="14.605" x2="43.18" y2="22.225" width="0.254" layer="16"/>
+<wire x1="50.8" y1="14.605" x2="44.45" y2="20.955" width="0.254" layer="16"/>
 <wire x1="53.34" y1="14.605" x2="50.8" y2="14.605" width="0.254" layer="1"/>
 <wire x1="62.23" y1="14.605" x2="53.34" y2="14.605" width="0.254" layer="16"/>
@@
 <via x="53.34" y="14.605" extent="1-16" drill="0.6"/>
 <via x="62.23" y="14.605" extent="1-16" drill="0.6"/>
+<wire x1="38.1" y1="28.575" x2="36.83" y2="29.845" width="0.254" layer="16"/>
+<wire x1="38.1" y1="22.225" x2="38.1" y2="28.575" width="0.254" layer="16"/>
+<wire x1="39.37" y1="20.955" x2="38.1" y2="22.225" width="0.254" layer="16"/>
+<wire x1="44.45" y1="20.955" x2="39.37" y2="20.955" width="0.254" layer="16"/>
 </signal>
 <signal name="N$24">

Commit message: Finished routing
Parts:
- S2: device SparkFun-Retired:SJ_2S-TRACE-PTH -> YMSynth:1X02
Routing:
- net GND: track 435.7 -> 0.00 mm, vias 2 -> 0
- net VCC: track 180.6 -> 248.8 mm, vias 1 -> 0
- net N$7: track 0.00 -> 62.9 mm, vias 0 -> 1
- net N$6: track 0.00 -> 60.0 mm, vias 0 -> 1
- net /RST: track 13.8 -> 73.3 mm, vias 0 -> 3
- net 1MHZE: track 47.3 -> 94.0 mm, vias 2 -> 4
- net R/W: track 49.5 -> 95.1 mm
- net A0: track 23.9 -> 63.8 mm, vias 0 -> 1
- net D0: track 36.1 -> 68.9 mm
- net /PGFC: track 33.1 -> 58.0 mm, vias 0 -> 2
- net YM/IRQ: track 88.6 -> 68.3 mm
- net AUDIO: track 64.1 -> 79.8 mm
- net N$2: track 28.1 -> 39.9 mm
- net N$8: track 57.5 -> 48.9 mm, vias 4 -> 1
- net N$14: track 35.0 -> 26.7 mm
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- added copper zone on layer 1, net GND
- added copper zone on layer 16, net GND
