File: eagle/BeebOPL.sch (EAGLE design)
At the start: 44 parts, among them IC1 LM324N, IC2 YM3014B, IC3 LM7805, IC5 74LS02N, IC6 YM3812, IC7 74LS04N, IC9 74HCT688N, J1 1 MHz Bus, J2 Feed-through, J3 3.5mm Jack, J4 DC-IN

Commit message: Added silkscreen
Parts:
- removed JP5: PWR, pinhead:PINHD-1X4
- added J6: 3.5mm Jack, SparkFun-Connectors:AUDIO-JACKPTH
- added LOGO1: OSHW-LOGO-BOTTOML, YMSynth:OSHW-LOGO-BOTTOML
- C1: value 4.7uF 35V -> 82pF; device resistor:CPOL-EUE2-5 -> resistor:C-EU050-024X044
- C10: value 100nF -> 220pF
- C11: value 100nF -> 4.7uF 35V; device resistor:C-EU050-024X044 -> YMSynth:CPOL-EUE2.5-5
- C2: value 470pF -> 4.7nF
- C3: value 10uF 16V -> 10nF; device resistor:CPOL-EUE2-5 -> resistor:C-EU050-024X044
- C4: value 220pF -> 100nF
- C5: value 82pF -> 100nF
- C6: device resistor:CPOL-EUE2-5 -> YMSynth:CPOL-EUE2.5-5
- C8: value 10nF -> 10uF 16V; device resistor:C-EU050-024X044 -> YMSynth:CPOL-EUE2.5-5
- C9: value 4.7nF -> 470pF
- IC1: value LM324N -> 74LS02N; device linear:LM324N -> 74xx-us:74LS02N
- IC2: value YM3014B -> LM7805; device YMSynth:YM3014B-DIP8 -> linear:7805TV
- IC3: value LM7805 -> 74LS04N; device linear:7805TV -> 74xx-us:74LS04N
- IC5: value 74LS02N -> YM3812; device 74xx-us:74LS02N -> YMSynth:YM3812-DIP24
- IC6: value YM3812 -> LM324N; device YMSynth:YM3812-DIP24 -> linear:LM324N
- IC7: value 74LS04N -> YM3014B; device 74xx-us:74LS04N -> YMSynth:YM3014B-DIP8
- J3: value 3.5mm Jack -> DC in; device SparkFun-Connectors:AUDIO-JACKPTH -> SparkFun-Connectors:POWER_JACKSLT
- J4: value DC-IN -> PWR; device SparkFun-Connectors:POWER_JACKSLT -> pinhead:PINHD-1X4
- J7: value AUDIO -> Audio
- R1: value 4k7 -> 470R
- R2: value 27k -> 470R
- R3: value 15k -> 470R
- R6: value 4k7 -> 15k
- R7: value 470R -> 27k
- R8, R9: value 470R -> 4k7
- RN1, RN2, RN3, RN4: value 2k2 -> 2k2 x 8
- S1: value 1MHz Bus Audio -> IRQ enable; device SparkFun-Retired:JUMPER-2PTH -> YMSynth:JUMPER-2PTH
- S2: value IRQ -> pwr sel; device YMSynth:JUMPER-2PTH -> YMSynth:J2
- S3: value REG -> 1MHz Bus Audio; device YMSynth:J2 -> SparkFun-Retired:JUMPER-2PTH
- renumbered IC9 to IC4, JP3 to J7, JP4 to J5, XTAL1 to Q1
Connections:
- net +12V: now also IC2.VI, J4.1, S2.3; no longer IC3.VI, JP5.1, S3.3
- net +5V: now also IC2.VO, J4.4, S2.1; no longer IC3.VO, JP5.4, S3.1
- net /IRQ: now also S1.1; no longer S2.1
- net /PGFC: now also IC1A.I1, IC1C.I1; no longer IC5A.I1, IC5C.I1
- net /RST: now also IC5./IC; no longer IC6./IC
- net 1MHZE: now also IC1A.I0, IC3C.I; no longer IC5A.I0, IC7C.I
- net A0: now also IC5.A0; no longer IC6.A0
- net AUDIO: now also S3.2; no longer S1.2
- net AUDIO_OUT: now also C11.-, J6.LEFT, J6.RIGHT, S3.1; no longer C1.-, J3.LEFT, J3.RIGHT, S1.1
- net CNPGFC: now also IC1B.O, IC1C.I0; no longer IC5B.O, IC5C.I0
- net D0: now also IC5.D0; no longer IC6.D0
- net D1: now also IC5.D1; no longer IC6.D1
- net D2: now also IC5.D2; no longer IC6.D2
- net D3: now also IC5.D3; no longer IC6.D3
- net D4: now also IC5.D4; no longer IC6.D4
- net D5: now also IC5.D5; no longer IC6.D5
- net D6: now also IC5.D6; no longer IC6.D6
- net D7: now also IC5.D7; no longer IC6.D7
- net DC: now also J3.PWR, S2.2; no longer J4.PWR, S3.2
- net GND: now also C1.2, C3.2, C8.-, IC1P.GND, IC3P.GND, IC5.GND, IC6P.V-, IC7.GND, J3.GND, J3.GNDBREAK, J4.2, J4.3, J6.SLEEVE, R8.1, R9.1; no longer C11.2, C3.-, C8.2, IC1P.V-, IC3.GND, IC5P.GND, IC6.GND, IC7P.GND, J3.SLEEVE, J4.GND, J4.GNDBREAK, JP5.2, JP5.3, R1.1, R6.1
- net N$1: now also C2.1, IC3A.O, R1.2; no longer C9.1, IC7A.O, R7.2
- net N$10: now also IC1A.O, IC1B.I0; no longer IC5A.O, IC5B.I0
- net N$11: now also C8.+, IC6D.+IN, IC7.RB; no longer C3.+, IC1D.+IN, IC2.RB
- net N$12: now also IC1B.I1, IC1C.O; no longer IC5B.I1, IC5C.O
- net N$13: now also IC6D.-IN, IC6D.OUT, IC7.MP, R8.2; no longer IC1D.-IN, IC1D.OUT, IC2.MP, R3.2
- net N$14: now also IC3D.O, IC5./RD; no longer IC6./RD, IC7D.O
- net N$15: now also IC6B.-IN, R6.1, R7.1; no longer IC1B.-IN, R2.1, R3.1
- net N$16: now also C11.+, IC6B.OUT, R7.2, R9.2; no longer C1.+, IC1B.OUT, R1.2, R2.2
- net N$18: now also IC6A.+IN, IC7.TOBUFF; no longer IC1A.+IN, IC2.TOBUFF
- net N$19: now also IC6A.-IN, IC6A.OUT, R4.1; no longer IC1A.-IN, IC1A.OUT, R5.1
- net N$2: now also IC1D.O, IC3B.I; no longer IC5D.O, IC7B.I
- net N$20: now also C9.1, R4.2, R5.1; no longer C2.1, R4.1, R5.2
- net N$21: now also C10.1, IC6C.+IN, R5.2; no longer C4.1, IC1C.+IN, R4.2
- net N$22: now also C9.2, IC6B.+IN, IC6C.-IN, IC6C.OUT; no longer C2.2, IC1B.+IN, IC1C.-IN, IC1C.OUT
- net N$23: now also IC5./CS; no longer IC6./CS
- net N$24: now also IC3B.O, IC5./WR; no longer IC6./WR, IC7B.O
- net N$25: now also R3.1; no longer R9.1
- net N$26: now also IC3E.O, IC5.0M; no longer IC6.0M, IC7E.O
- net N$28: now also IC3E.I, IC3F.O, R2.2; no longer IC7E.I, IC7F.O, R8.2
- net N$3: now also IC1D.I0, IC3C.O; no longer IC5D.I0, IC7C.O
- net N$5: now also C2.2, IC3F.I, R2.1; no longer C9.2, IC7F.I, R8.1
- net N$6: now also IC5.SH, IC7.LOAD; no longer IC2.LOAD, IC6.SH
- net N$7: now also IC5.MO, IC7.SD; no longer IC2.SD, IC6.MO
- net N$8: now also IC5.0SY, IC7.CLOCK; no longer IC2.CLOCK, IC6.0SY
- net N$9: now also C1.1, IC3A.I, R1.1; no longer C5.1, IC7A.I, R7.1
- net R/W: now also IC1D.I1, IC3D.I; no longer IC5D.I1, IC7D.I
- net VCC: now also C3.1, C4.1, C5.1, IC1P.VCC, IC3P.VCC, IC5.VSS, IC6P.V+, IC7.VDD, R3.2; no longer C10.1, C11.1, C8.1, IC1P.V+, IC2.VDD, IC5P.VCC, IC6.VSS, IC7P.VCC, R9.2
- net YM/IRQ: now also IC5./IRQ, S1.2; no longer IC6./IRQ, S2.2
Other:
- note added: "DATE: 1 October 2016"
- note added: "REVISION: 1.00"
- note added: "Robert Lazarus https://github.com/lazarusr/beebopl"
- note removed: "Bob's board (text behind YM3812)"
- note removed: "Check that sockets etc fit with overhang"
- note removed: "Check the pinout orientation for power connector"
- note removed: "Check whether I want to change the footprint of the 3.5mm connector"
- note removed: "DATE: 29 Sept 2016"
- note removed: "IMPORTANT – Check board for links at: 3 pin jumper MOSFET IRQ jumper"
- note removed: "Put arrows at track cut points"
- note removed: "REVISION: 0.90"
- note removed: "To do"
- moved on the sheet: C10, C2, C4, C5, C7, C9, J1, J2, R1, R2, R3, R4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

Commit message: Final board sent to fab
Parts:
- IC7: value YM3014B -> Y3014B
Other:
- note added: "DATE: 2 October 2016"
- note removed: "DATE: 1 October 2016"
Changed lines of the file:
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@@
 <part name="GND5" library="supply1" deviceset="GND" device=""/>
 <part name="Q1" library="special" deviceset="XTAL/S" device="" value="3.579MHz"/>
-<part name="IC7" library="YMSynth" deviceset="YM3014B" device="-DIP8" value="YM3014B"/>
+<part name="IC7" library="YMSynth" deviceset="YM3014B" device="-DIP8" value="Y3014B"/>
 <part name="GND14" library="supply1" deviceset="GND" device=""/>
 <part name="P+16" library="supply1" deviceset="VCC" device=""/>
@@
 <text x="-175.26" y="-152.4" size="10.16" layer="97" font="vector">REVISION: 1.00</text>
 <wire x1="-182.88" y1="-180.34" x2="2.54" y2="-180.34" width="0.1524" layer="97"/>
-<text x="-175.26" y="-175.26" size="10.16" layer="97" font="vector">DATE: 1 October 2016</text>
+<text x="-175.26" y="-175.26" size="10.16" layer="97" font="vector">DATE: 2 October 2016</text>
 <text x="-96.52" y="-50.8" size="1.778" layer="97" rot="R90">Divide track to use
 12v from power jack</text>
